Commit message: sec com

File: tags_in_urdf/urdf/box.xacro (robot description, xacro)
@@ -50,5 +50,5 @@
     <parent link="box"/>
     <child link="artag4"/>
-    <origin rpy="0 0 0" xyz="0 0 0.2"/>
+    <origin rpy="0 0 0" xyz="0 0 0.025"/>
     <!-- <origin rpy="0 0 -1.571" xyz="0 0 0"/> -->
   </joint>

Commit message: a

File: tags_in_urdf/urdf/box.xacro (robot description, xacro)
@@ -1,11 +1,10 @@
 <?xml version="1.0"?>
 <robot name="box" xmlns:xacro="http://ros.org/wiki/xacro">
-  <link name="box_world"/>
-<!--Box with button-->
+  <xacro:property name="tag" value="tag.dae" />
   <link name="box">
     <visual>
       <origin rpy="0 0 0" xyz="0 0 0"/>
       <geometry>
-        <box size="0.2 0.2 0.05"/>
+        <box size="0.1 0.1 0.1"/>
       </geometry>
     </visual>
@@ -13,5 +12,5 @@
       <origin rpy="0 0 0" xyz="0 0 0"/>
       <geometry>
-        <box size="0.2 0.2 0.05"/>
+        <box size="0.1 0.1 0.1"/>
       </geometry>
     </collision>
@@ -22,15 +21,9 @@
     </inertial>
   </link>
-  <joint name="box_joint" type="fixed">
-    <parent link="box_world"/>
-    <child link="box"/>
-    <!-- <origin rpy="0 0 3.14" xyz="-0.35 0 0.2"/> -->
-    <origin rpy="0 0 3.14" xyz="0 0 0"/>
-  </joint>
   <link name="artag4">
     <visual>
       <origin rpy="0 0 0" xyz="0 0 0"/>
       <geometry>
-        <mesh filename="package://tags_in_urdf/meshes/tag.dae"/>
+        <mesh filename="package://tags_in_urdf/meshes/${tag}"/>
       </geometry>
     </visual>
@@ -38,5 +31,5 @@
       <origin rpy="0 0 0" xyz="0 0 0"/>
       <geometry>
-        <mesh filename="package://tags_in_urdf/meshes/tag.dae"/>
+        <mesh filename="package://tags_in_urdf/meshes/${tag}"/>
       </geometry>
     </collision>
@@ -50,13 +43,5 @@
     <parent link="box"/>
     <child link="artag4"/>
-    <origin rpy="0 0 0" xyz="0 0 0.025"/>
-    <!-- <origin rpy="0 0 -1.571" xyz="0 0 0"/> -->
+    <origin rpy="0 0 0" xyz="0 1 1"/>
   </joint>
-  <!-- <link name="button"/>
-  <joint name="button" type="fixed">
-    <parent link="artag4"/>
-    <child link="button"/>
-    <origin rpy="3.14 1.5708 3.14" xyz="0.12 0.0 0.07"/>
-    <origin rpy="0 0 0" xyz="0 -0.11500000 0.02361546"/>
-  </joint> -->
 </robot>
